Commit message: Complete autonomous navigation, mapping, and kinematic gait engine updates

File: src/phantomx_description/urdf/phantomx.urdf (robot description, URDF)
Before this commit: robot PhantomX, 26 links, 25 joints
Joints:
- joint j_c1_lf: limit lower=-2.6179939 upper=2.6179939 effort=2.8 velocity=5.6548668 -> lower=-3.14159 upper=3.14159 effort=2.8 velocity=5.6548668
- joint j_c1_lm: limit lower=-2.6179939 upper=2.6179939 effort=2.8 velocity=5.6548668 -> lower=-3.14159 upper=3.14159 effort=2.8 velocity=5.6548668
- joint j_c1_lr: limit lower=-2.6179939 upper=2.6179939 effort=2.8 velocity=5.6548668 -> lower=-3.14159 upper=3.14159 effort=2.8 velocity=5.6548668
- joint j_c1_rf: limit lower=-2.6179939 upper=2.6179939 effort=2.8 velocity=5.6548668 -> lower=-3.14159 upper=3.14159 effort=2.8 velocity=5.6548668
- joint j_c1_rm: limit lower=-2.6179939 upper=2.6179939 effort=2.8 velocity=5.6548668 -> lower=-3.14159 upper=3.14159 effort=2.8 velocity=5.6548668
- joint j_c1_rr: limit lower=-2.6179939 upper=2.6179939 effort=2.8 velocity=5.6548668 -> lower=-3.14159 upper=3.14159 effort=2.8 velocity=5.6548668
- joint j_thigh_lf: limit lower=-2.6179939 upper=2.6179939 effort=2.8 velocity=5.6548668 -> lower=-3.14159 upper=3.14159 effort=2.8 velocity=5.6548668
- joint j_thigh_lm: limit lower=-2.6179939 upper=2.6179939 effort=2.8 velocity=5.6548668 -> lower=-3.14159 upper=3.14159 effort=2.8 velocity=5.6548668
- joint j_thigh_lr: limit lower=-2.6179939 upper=2.6179939 effort=2.8 velocity=5.6548668 -> lower=-3.14159 upper=3.14159 effort=2.8 velocity=5.6548668
- joint j_thigh_rf: limit lower=-2.6179939 upper=2.6179939 effort=2.8 velocity=5.6548668 -> lower=-3.14159 upper=3.14159 effort=2.8 velocity=5.6548668
- joint j_thigh_rm: limit lower=-2.6179939 upper=2.6179939 effort=2.8 velocity=5.6548668 -> lower=-3.14159 upper=3.14159 effort=2.8 velocity=5.6548668
- joint j_thigh_rr: limit lower=-2.6179939 upper=2.6179939 effort=2.8 velocity=5.6548668 -> lower=-3.14159 upper=3.14159 effort=2.8 velocity=5.6548668
- joint j_tibia_lf: limit lower=-2.6179939 upper=2.6179939 effort=2.8 velocity=5.6548668 -> lower=-3.14159 upper=3.14159 effort=2.8 velocity=5.6548668
- joint j_tibia_lm: limit lower=-2.6179939 upper=2.6179939 effort=2.8 velocity=5.6548668 -> lower=-3.14159 upper=3.14159 effort=2.8 velocity=5.6548668
- joint j_tibia_lr: limit lower=-2.6179939 upper=2.6179939 effort=2.8 velocity=5.6548668 -> lower=-3.14159 upper=3.14159 effort=2.8 velocity=5.6548668
- joint j_tibia_rf: limit lower=-2.6179939 upper=2.6179939 effort=2.8 velocity=5.6548668 -> lower=-3.14159 upper=3.14159 effort=2.8 velocity=5.6548668
- joint j_tibia_rm: limit lower=-2.6179939 upper=2.6179939 effort=2.8 velocity=5.6548668 -> lower=-3.14159 upper=3.14159 effort=2.8 velocity=5.6548668
- joint j_tibia_rr: limit lower=-2.6179939 upper=2.6179939 effort=2.8 velocity=5.6548668 -> lower=-3.14159 upper=3.14159 effort=2.8 velocity=5.6548668
